Commit message: ex01 fixed

File: Mod5/ex01/robot.urdf (robot description, URDF)
Before this commit: robot sam_bot, 3 links, 2 joints
Links:
- removed link base_footprint
- removed link front_caster
- added link wheel_left_link; visual cylinder length=0.1 radius=0.2
- added link wheel_right_link; visual cylinder length=0.1 radius=0.2
- link base_link: geometry visual box size=0.7 0.4 0.2
Joints:
- removed joint base_joint
- removed joint caster_joint
- added joint wheel_left_joint: type continuous, parent base_link, child wheel_left_link, origin xyz=0.25 0.2 -0.05, axis 0 1 0
- added joint wheel_right_joint: type continuous, parent base_link, child wheel_right_link, origin xyz=0.25 -0.2 -0.05, axis 0 1 0
